File: KalyPCB/KalyPCB.kicad_pcb (KiCad board)
At the start: 2 copper layers, 135.6 x 99.8 mm, 26 parts, among them J1 TRRS

Commit message: Remove text and images from PCB
Parts:
- removed G*** (x3): LOGO, LOGO
Other:
- board text removed: "By: Kael S.A."
- board text removed: "Kaly42"
- board text removed: "Kaly42 V1"
- board text removed: "https://github.com/Dwctor/Kaly"
